File: KiCAD/EBS.kicad_pcb (KiCad board)
At the start: 2 copper layers, 44.4 x 27.4 mm, 21 parts, among them Q1 BC547, Q2 BC557

Commit message: Update
Routing:
- added copper zone on B.Cu, net GND
- removed copper zone on F.Cu, net GND
